File: trinamic_wiring/tmc2209_bidirectional_coupled.kicad_sch (KiCad schematic)
At the start: 3 parts

Commit message: Redo schematic symbols
Parts:
- removed TMC?: TMC2209, symbol Janelia:SIMPLIFIED_TMC2209_UART
- removed microcontroller?: microcontroller, symbol Janelia:SIMPLIFIED_MCU_UART
- added MICROCONTROLLER4: DOC_MCU_UART, symbol Janelia:DOC_MCU_UART
- added TMC6: DOC_TMC2209, symbol Janelia:DOC_TMC2209
Connections:
- net at R2.1: now also MICROCONTROLLER4.1 (TX)
Changed lines of the file:
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@@
     (company "Janelia Research Campus")
   )
-  (junction (at 102.87 106.68) (diameter 0) (color 0 0 0 0)
-  )
-  (wire (pts (xy 102.87 87.63) (xy 102.87 90.17))
+  (wire (pts (xy 127 88.9) (xy 129.54 88.9))
     (stroke (width 0) (type default))
   )
-  (wire (pts (xy 138.43 80.01) (xy 138.43 106.68))
-    (stroke (width 0) (type default))
-  )
-  (wire (pts (xy 102.87 106.68) (xy 138.43 106.68))
-    (stroke (width 0) (type default))
-  )
-  (wire (pts (xy 102.87 102.87) (xy 102.87 106.68))
-    (stroke (width 0) (type default))
-  )
-  (wire (pts (xy 100.33 87.63) (xy 102.87 87.63))
-    (stroke (width 0) (type default))
-  )
-  (wire (pts (xy 100.33 106.68) (xy 102.87 106.68))
-    (stroke (width 0) (type default))
-  )
-  (symbol (lib_id "Janelia:SIMPLIFIED_MCU_UART") (at 87.63 96.52 0) (unit 1)
-    (in_bom yes) (on_board yes) (dnp no)
-    (property "Reference" "microcontroller?" (at 87.63 96.52 0) (do_not_autoplace)
+  (symbol (lib_id "Janelia:DOC_TMC2209") (at 165.1 99.06 0) (unit 1)
+    (in_bom yes) (on_board yes) (dnp no) (fields_autoplaced)
+    (property "Reference" "TMC6" (at 165.1 80.01 0)
+      (effects (font (size 1.27 1.27)) hide)
+    )
+    (property "Value" "DOC_TMC2209" (at 165.1 85.09 0)
       (effects (font (size 1.524 1.524)) hide)
     )
-    (property "Value" "microcontroller" (at 87.63 96.52 0)
-      (effects (font (size 1.524 1.524)))
-    )
-    (property "Footprint" "" (at 85.09 123.19 0)
+    (property "Footprint" "" (at 162.56 125.73 0)
       (effects (font (size 1.524 1.524)) hide)
     )
-    (property "Datasheet" "" (at 87.63 96.52 0)
+    (property "Datasheet" "" (at 165.1 99.06 0)
       (effects (font (size 1.524 1.524)) hide)
+    )
+    (property "Sim.Enable" "0" (at 165.1 82.55 0)
+      (effects (font (size 1.27 1.27)) hide)
+    )
+    (pin "0")
+    (pin "1")
+    (pin "10")
+    (pin "2")
+    (pin "3")
+    (pin "4")
+    (pin "5")
+    (pin "6")
+    (pin "7")
+    (pin "8")
+    (pin "9")
+    (instances
+      (project "trinamic_wiring"
+        (path "/e4144788-6304-493f-818e-5d881d3b7418/c8eda2b5-ab13-4033-82d9-875c9fcaf884/13e2a7b5-46df-44bb-8dde-5d79d190b8bf"
+          (reference "TMC6") (unit 1)
+        )
+        (path "/e4144788-6304-493f-818e-5d881d3b7418/c8eda2b5-ab13-4033-82d9-875c9fcaf884/e3613d8e-f506-47d6-ad2d-b0f5798d9847"
+          (reference "TMC7") (unit 1)
+        )
+      )
+    )
+  )
+  (symbol (lib_id "Janelia:DOC_MCU_UART") (at 114.3 99.06 0) (unit 1)
+    (in_bom yes) (on_board yes) (dnp no) (fields_autoplaced)
+    (property "Reference" "MICROCONTROLLER4" (at 114.3 80.01 0) (do_not_autoplace)
+      (effects (font (size 1.27 1.27)) hide)
+    )
+    (property "Value" "DOC_MCU_UART" (at 114.3 85.09 0)
+      (effects (font (size 1.524 1.524)) hide)
+    )
+    (property "Footprint" "" (at 111.76 125.73 0)
+      (effects (font (size 1.524 1.524)) hide)
+    )
+    (property "Datasheet" "" (at 114.3 99.06 0)
+      (effects (font (size 1.524 1.524)) hide)
+    )
+    (property "Sim.Enable" "0" (at 114.3 82.55 0)
+      (effects (font (size 1.27 1.27)) hide)
     )
     (pin "0")
@@
       (project "trinamic_wiring"
         (path "/e4144788-6304-493f-818e-5d881d3b7418/c8eda2b5-ab13-4033-82d9-875c9fcaf884/13e2a7b5-46df-44bb-8dde-5d79d190b8bf"
-          (reference "microcontroller?") (unit 1)
+          (reference "MICROCONTROLLER4") (unit 1)
         )
         (path "/e4144788-6304-493f-818e-5d881d3b7418/c8eda2b5-ab13-4033-82d9-875c9fcaf884/e3613d8e-f506-47d6-ad2d-b0f5798d9847"
-          (reference "microcontroller1") (unit 1)
-        )
-        (path "/e4144788-6304-493f-818e-5d881d3b7418/c8eda2b5-ab13-4033-82d9-875c9fcaf884/5f6f310d-167d-42a3-8815-1b623fe73dc8"
-          (reference "microcontroller2") (unit 1)
+          (reference "MICROCONTROLLER5") (unit 1)
         )
       )
     )
   )
-  (symbol (lib_id "Janelia:SIMPLIFIED_TMC2209_UART") (at 138.43 64.77 0) (unit 1)
-    (in_bom yes) (on_board yes) (dnp no) (fields_autoplaced)
-    (property "Reference" "TMC?" (at 138.43 64.77 0) (do_not_autoplace)
+  (symbol (lib_id "Janelia:R_1k_0402") (at 135.89 88.9 90) (unit 1)
+    (in_bom yes) (on_board yes) (dnp no)
+    (property "Reference" "R2" (at 135.89 87.63 0)
+      (effects (font (size 1.016 1.016)) (justify left) hide)
+    )
+    (property "Value" "1k" (at 135.89 88.9 90)
+      (effects (font (size 0.762 0.762)))
+    )
+    (property "Footprint" "Janelia:R_0402_1005Metric" (at 135.89 90.678 90)
+      (effects (font (size 0.762 0.762)) hide)
+    )
+    (property "Datasheet" "" (at 135.89 86.868 90)
+      (effects (font (size 0.762 0.762)))
+    )
+    (property "Vendor" "Digi-Key" (at 133.35 84.328 90)
       (effects (font (size 1.524 1.524)) hide)
     )
-    (property "Value" "TMC2209" (at 138.43 64.77 0)
-      (effects (font (size 1.524 1.524)))
-    )
-    (property "Footprint" "" (at 135.89 91.44 0)
+    (property "Vendor Part Number" "311-1.00KLRCT-ND" (at 130.81 81.788 90)
       (effects (font (size 1.524 1.524)) hide)
     )
-    (property "Datasheet" "" (at 138.43 64.77 0)
+    (property "Description" "RES SMD 1K OHM 1% 1/16W" (at 128.27 79.248 90)
       (effects (font (size 1.524 1.524)) hide)
     )
-    (pin "0")
-    (instances
-      (project "trinamic_wiring"
-        (path "/e4144788-6304-493f-818e-5d881d3b7418/c8eda2b5-ab13-4033-82d9-875c9fcaf884/13e2a7b5-46df-44bb-8dde-5d79d190b8bf"
-          (reference "TMC?") (unit 1)
-        )
-        (path "/e4144788-6304-493f-818e-5d881d3b7418/c8eda2b5-ab13-4033-82d9-875c9fcaf884/e3613d8e-f506-47d6-ad2d-b0f5798d9847"
-          (reference "TMC1") (unit 1)
-        )
-        (path "/e4144788-6304-493f-818e-5d881d3b7418/c8eda2b5-ab13-4033-82d9-875c9fcaf884/5f6f310d-167d-42a3-8815-1b623fe73dc8"
-          (reference "TMC2") (unit 1)
-        )
-      )
-    )
-  )
-  (symbol (lib_id "Janelia:R_1k_0402") (at 102.87 96.52 0) (unit 1)
-    (in_bom yes) (on_board yes) (dnp no)
-    (property "Reference" "R2" (at 104.14 96.52 0)
-      (effects (font (size 1.016 1.016)) (justify left) hide)
-    )
-    (property "Value" "1k" (at 102.87 96.52 90)
-      (effects (font (size 0.762 0.762)))
-    )
-    (property "Footprint" "Janelia:R_0402_1005Metric" (at 101.092 96.52 90)
-      (effects (font (size 0.762 0.762)) hide)
-    )
-    (property "Datasheet" "" (at 104.902 96.52 90)
-      (effects (font (size 0.762 0.762)))
-    )
-    (property "Vendor" "Digi-Key" (at 107.442 93.98 90)
-      (effects (font (size 1.524 1.524)) hide)
-    )
-    (property "Vendor Part Number" "311-1.00KLRCT-ND" (at 109.982 91.44 90)
-      (effects (font (size 1.524 1.524)) hide)
-    )
-    (property "Description" "RES SMD 1K OHM 1% 1/16W" (at 112.522 88.9 90)
-      (effects (font (size 1.524 1.524)) hide)
-    )
-    (property "Package" "0402" (at 102.87 96.52 0)
+    (property "Package" "0402" (at 135.89 88.9 0)
       (effects (font (size 1.27 1.27)) hide)
     )
-    (property "Manufacturer" "YAGEO" (at 102.87 96.52 0)
+    (property "Manufacturer" "YAGEO" (at 135.89 88.9 0)
       (effects (font (size 1.27 1.27)) hide)
     )
-    (property "Manufacturer Part Number" "RC0402FR-071KL" (at 102.87 96.52 0)
+    (property "Manufacturer Part Number" "RC0402FR-071KL" (at 135.89 88.9 0)
       (effects (font (size 1.27 1.27)) hide)
     )
