File: trinamic_wiring/tmc2209_unidirectional_serial_address.kicad_sch (KiCad schematic)
At the start: 3 parts

Commit message: Redo schematic symbols
Parts:
- added MICROCONTROLLER4: DOC_MCU_UART, symbol Janelia:DOC_MCU_UART
- added TMC6 (x2): DOC_TMC2209, symbol Janelia:DOC_TMC2209
Connections:
- net +VCCIO: now also TMC6.9 (AD0); no longer TMC3.2 (MS1_AD0)
- new net: MICROCONTROLLER4.1 (TX), TMC6.0 (UART), TMC6.0 (UART)
- no-connect marks 4 -> 8
Changed lines of the file:
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@@
   (junction (at 138.43 87.63) (diameter 0) (color 0 0 0 0)
+  )
+  (junction (at 161.29 101.6) (diameter 0) (color 0 0 0 0)
   )
   (no_connect (at 133.35 80.01))
   (no_connect (at 130.81 80.01))
+  (no_connect (at 163.83 116.84))
+  (no_connect (at 163.83 114.3))
+  (no_connect (at 138.43 121.92))
+  (no_connect (at 163.83 144.78))
   (no_connect (at 156.21 80.01))
   (no_connect (at 100.33 106.68))
+  (wire (pts (xy 161.29 101.6) (xy 161.29 129.54))
+    (stroke (width 0) (type default))
+  )
   (wire (pts (xy 138.43 87.63) (xy 161.29 87.63))
     (stroke (width 0) (type default))
@@
     (stroke (width 0) (type default))
   )
+  (wire (pts (xy 138.43 101.6) (xy 161.29 101.6))
+    (stroke (width 0) (type default))
+  )
   (wire (pts (xy 153.67 80.01) (xy 153.67 82.55))
     (stroke (width 0) (type default))
   )
+  (wire (pts (xy 161.29 142.24) (xy 163.83 142.24))
+    (stroke (width 0) (type default))
+  )
+  (wire (pts (xy 161.29 129.54) (xy 163.83 129.54))
+    (stroke (width 0) (type default))
+  )
+  (wire (pts (xy 161.29 101.6) (xy 163.83 101.6))
+    (stroke (width 0) (type default))
+  )
   (wire (pts (xy 138.43 80.01) (xy 138.43 87.63))
     (stroke (width 0) (type default))
@@
     (stroke (width 0) (type default))
   )
-  (label "+VCCIO" (at 153.67 82.55 180) (fields_autoplaced)
+  (label "+VCCIO" (at 161.29 142.24 180) (fields_autoplaced)
     (effects (font (size 1.27 1.27) (color 255 0 255 1)) (justify right bottom))
+  )
+  (symbol (lib_id "Janelia:DOC_MCU_UART") (at 125.73 111.76 0) (unit 1)
+    (in_bom yes) (on_board yes) (dnp no) (fields_autoplaced)
+    (property "Reference" "MICROCONTROLLER4" (at 125.73 92.71 0) (do_not_autoplace)
+      (effects (font (size 1.27 1.27)) hide)
+    )
+    (property "Value" "DOC_MCU_UART" (at 125.73 97.79 0)
+      (effects (font (size 1.524 1.524)) hide)
+    )
+    (property "Footprint" "" (at 123.19 138.43 0)
+      (effects (font (size 1.524 1.524)) hide)
+    )
+    (property "Datasheet" "" (at 125.73 111.76 0)
+      (effects (font (size 1.524 1.524)) hide)
+    )
+    (property "Sim.Enable" "0" (at 125.73 95.25 0)
+      (effects (font (size 1.27 1.27)) hide)
+    )
+    (pin "0")
+    (pin "1")
+    (instances
+      (project "trinamic_wiring"
+        (path "/e4144788-6304-493f-818e-5d881d3b7418/c8eda2b5-ab13-4033-82d9-875c9fcaf884/13e2a7b5-46df-44bb-8dde-5d79d190b8bf"
+          (reference "MICROCONTROLLER4") (unit 1)
+        )
+        (path "/e4144788-6304-493f-818e-5d881d3b7418/c8eda2b5-ab13-4033-82d9-875c9fcaf884/5b0a2695-6b0b-4c82-b9d6-7e19fee75501"
+          (reference "MICROCONTROLLER1") (unit 1)
+        )
+        (path "/e4144788-6304-493f-818e-5d881d3b7418/c8eda2b5-ab13-4033-82d9-875c9fcaf884/a2ce530e-f5b5-4e3e-9188-e4bc8f84c739"
+          (reference "MICROCONTROLLER3") (unit 1)
+        )
+      )
+    )
   )
   (symbol (lib_id "Janelia:SIMPLIFIED_MCU_UART") (at 87.63 96.52 0) (unit 1)
@@
     )
   )
+  (symbol (lib_id "Janelia:DOC_TMC2209") (at 176.53 139.7 0) (unit 1)
+    (in_bom yes) (on_board yes) (dnp no) (fields_autoplaced)
+    (property "Reference" "TMC6" (at 176.53 120.65 0)
+      (effects (font (size 1.27 1.27)) hide)
+    )
+    (property "Value" "DOC_TMC2209" (at 176.53 125.73 0)
+      (effects (font (size 1.524 1.524)) hide)
+    )
+    (property "Footprint" "" (at 173.99 166.37 0)
+      (effects (font (size 1.524 1.524)) hide)
+    )
+    (property "Datasheet" "" (at 176.53 139.7 0)
+      (effects (font (size 1.524 1.524)) hide)
+    )
+    (property "Sim.Enable" "0" (at 176.53 123.19 0)
+      (effects (font (size 1.27 1.27)) hide)
+    )
+    (pin "0")
+    (pin "1")
+    (pin "10")
+    (pin "2")
+    (pin "3")
+    (pin "4")
+    (pin "5")
+    (pin "6")
+    (pin "7")
+    (pin "8")
+    (pin "9")
+    (instances
+      (project "trinamic_wiring"
+        (path "/e4144788-6304-493f-818e-5d881d3b7418/c8eda2b5-ab13-4033-82d9-875c9fcaf884/13e2a7b5-46df-44bb-8dde-5d79d190b8bf"
+          (reference "TMC6") (unit 1)
+        )
+        (path "/e4144788-6304-493f-818e-5d881d3b7418/c8eda2b5-ab13-4033-82d9-875c9fcaf884/5b0a2695-6b0b-4c82-b9d6-7e19fee75501"
+          (reference "TMC8") (unit 1)
+        )
+        (path "/e4144788-6304-493f-818e-5d881d3b7418/c8eda2b5-ab13-4033-82d9-875c9fcaf884/a2ce530e-f5b5-4e3e-9188-e4bc8f84c739"
+          (reference "TMC5") (unit 1)
+        )
+      )
+    )
+  )
   (symbol (lib_id "Janelia:SIMPLIFIED_TMC2209_ADDRESSES") (at 138.43 64.77 0) (unit 1)
     (in_bom yes) (on_board yes) (dnp no)
@@
         )
       )
+    )
+  )
+  (symbol (lib_name "DOC_TMC2209_1") (lib_id "Janelia:DOC_TMC2209") (at 176.53 111.76 0) (unit 1)
+    (in_bom yes) (on_board yes) (dnp no) (fields_autoplaced)
+    (property "Reference" "TMC6" (at 176.53 92.71 0)
+      (effects (font (size 1.27 1.27)) hide)
+    )
+    (property "Value" "DOC_TMC2209" (at 176.53 97.79 0)
+      (effects (font (size 1.524 1.524)) hide)
+    )
+    (property "Footprint" "" (at 173.99 138.43 0)
+      (effects (font (size 1.524 1.524)) hide)
+    )
+    (property "Datasheet" "" (at 176.53 111.76 0)
+      (effects (font (size 1.524 1.524)) hide)
+    )
+    (property "Sim.Enable" "0" (at 176.53 95.25 0)
+      (effects (font (size 1.27 1.27)) hide)
+    )
+    (pin "0")
+    (pin "1")
+    (pin "10")
+    (pin "2")
+    (pin "3")
+    (pin "4")
+    (pin "5")
+    (pin "6")
+    (pin "7")
+    (pin "8")
+    (pin "9")
+    (instances
+      (project "trinamic_wiring"
+        (path "/e4144788-6304-493f-818e-5d881d3b7418/c8eda2b5-ab13-4033-82d9-875c9fcaf884/13e2a7b5-46df-44bb-8dde-5d79d190b8bf"
+          (reference "TMC6") (unit 1)
+        )
+        (path "/e4144788-6304-493f-818e-5d881d3b7418/c8eda2b5-ab13-4033-82d9-875c9fcaf884/5b0a2695-6b0b-4c82-b9d6-7e19fee75501"
+          (reference "TMC1") (unit 1)
+        )
+        (path "/e4144788-6304-493f-818e-5d881d3b7418/c8eda2b5-ab13-4033-82d9-875c9fcaf884/a2ce530e-f5b5-4e3e-9188-e4bc8f84c739"
+          (reference "TMC4") (unit 1)
+        )
+      )
