File: trinamic_wiring/tmc2209_bidirectional_coupled_multiple_address.kicad_sch (KiCad schematic)
At the start: 4 parts

Commit message: Add TMC51X0 files
Parts:
- renumbered MICROCONTROLLER4 to MICROCONTROLLER7, R2 to R4, TMC6 to TMC11, TMC6 to TMC12
Changed lines of the file:
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@@
   (symbol (lib_name "DOC_TMC2209_1") (lib_id "Janelia:DOC_TMC2209") (at 166.37 87.63 0) (unit 1)
     (in_bom yes) (on_board yes) (dnp no) (fields_autoplaced)
-    (property "Reference" "TMC6" (at 166.37 68.58 0)
+    (property "Reference" "TMC11" (at 166.37 68.58 0)
       (effects (font (size 1.27 1.27)) hide)
     )
@@
     (instances
       (project "trinamic_wiring"
-        (path "/e4144788-6304-493f-818e-5d881d3b7418/c8eda2b5-ab13-4033-82d9-875c9fcaf884/13e2a7b5-46df-44bb-8dde-5d79d190b8bf"
-          (reference "TMC6") (unit 1)
-        )
-        (path "/e4144788-6304-493f-818e-5d881d3b7418/c8eda2b5-ab13-4033-82d9-875c9fcaf884/5b0a2695-6b0b-4c82-b9d6-7e19fee75501"
-          (reference "TMC1") (unit 1)
-        )
-        (path "/e4144788-6304-493f-818e-5d881d3b7418/c8eda2b5-ab13-4033-82d9-875c9fcaf884/a2ce530e-f5b5-4e3e-9188-e4bc8f84c739"
-          (reference "TMC4") (unit 1)
-        )
         (path "/e4144788-6304-493f-818e-5d881d3b7418/c8eda2b5-ab13-4033-82d9-875c9fcaf884/5f6f310d-167d-42a3-8815-1b623fe73dc8"
           (reference "TMC11") (unit 1)
         )
-        (path "/e4144788-6304-493f-818e-5d881d3b7418/c8eda2b5-ab13-4033-82d9-875c9fcaf884/00672f55-5cea-4051-abd7-9136695f76d0"
-          (reference "TMC2") (unit 1)
+        (path "/e4144788-6304-493f-818e-5d881d3b7418/a161638e-a96f-4455-865a-1d7502675f43/5f6f310d-167d-42a3-8815-1b623fe73dc8"
+          (reference "TMC6") (unit 1)
         )
       )
@@
   (symbol (lib_id "Janelia:DOC_TMC2209") (at 166.37 115.57 0) (unit 1)
     (in_bom yes) (on_board yes) (dnp no) (fields_autoplaced)
-    (property "Reference" "TMC6" (at 166.37 96.52 0)
+    (property "Reference" "TMC12" (at 166.37 96.52 0)
       (effects (font (size 1.27 1.27)) hide)
     )
@@
     (instances
       (project "trinamic_wiring"
-        (path "/e4144788-6304-493f-818e-5d881d3b7418/c8eda2b5-ab13-4033-82d9-875c9fcaf884/13e2a7b5-46df-44bb-8dde-5d79d190b8bf"
-          (reference "TMC6") (unit 1)
-        )
-        (path "/e4144788-6304-493f-818e-5d881d3b7418/c8eda2b5-ab13-4033-82d9-875c9fcaf884/5b0a2695-6b0b-4c82-b9d6-7e19fee75501"
-          (reference "TMC8") (unit 1)
-        )
-        (path "/e4144788-6304-493f-818e-5d881d3b7418/c8eda2b5-ab13-4033-82d9-875c9fcaf884/a2ce530e-f5b5-4e3e-9188-e4bc8f84c739"
-          (reference "TMC5") (unit 1)
-        )
         (path "/e4144788-6304-493f-818e-5d881d3b7418/c8eda2b5-ab13-4033-82d9-875c9fcaf884/5f6f310d-167d-42a3-8815-1b623fe73dc8"
           (reference "TMC12") (unit 1)
         )
-        (path "/e4144788-6304-493f-818e-5d881d3b7418/c8eda2b5-ab13-4033-82d9-875c9fcaf884/00672f55-5cea-4051-abd7-9136695f76d0"
-          (reference "TMC3") (unit 1)
+        (path "/e4144788-6304-493f-818e-5d881d3b7418/a161638e-a96f-4455-865a-1d7502675f43/5f6f310d-167d-42a3-8815-1b623fe73dc8"
+          (reference "TMC6") (unit 1)
         )
       )
@@
   (symbol (lib_id "Janelia:R_1k_0402") (at 134.62 77.47 90) (unit 1)
     (in_bom yes) (on_board yes) (dnp no)
-    (property "Reference" "R2" (at 134.62 76.2 0)
+    (property "Reference" "R4" (at 134.62 76.2 0)
       (effects (font (size 1.016 1.016)) (justify left) hide)
     )
@@
     (instances
       (project "trinamic_wiring"
-        (path "/e4144788-6304-493f-818e-5d881d3b7418/c8eda2b5-ab13-4033-82d9-875c9fcaf884/e3613d8e-f506-47d6-ad2d-b0f5798d9847"
-          (reference "R2") (unit 1)
-        )
         (path "/e4144788-6304-493f-818e-5d881d3b7418/c8eda2b5-ab13-4033-82d9-875c9fcaf884/5f6f310d-167d-42a3-8815-1b623fe73dc8"
           (reference "R4") (unit 1)
         )
-        (path "/e4144788-6304-493f-818e-5d881d3b7418/c8eda2b5-ab13-4033-82d9-875c9fcaf884/00672f55-5cea-4051-abd7-9136695f76d0"
-          (reference "R3") (unit 1)
+        (path "/e4144788-6304-493f-818e-5d881d3b7418/a161638e-a96f-4455-865a-1d7502675f43/5f6f310d-167d-42a3-8815-1b623fe73dc8"
+          (reference "R2") (unit 1)
         )
       )
@@
   (symbol (lib_id "Janelia:DOC_MCU") (at 113.03 87.63 0) (unit 1)
     (in_bom yes) (on_board yes) (dnp no) (fields_autoplaced)
-    (property "Reference" "MICROCONTROLLER4" (at 113.03 68.58 0)
+    (property "Reference" "MICROCONTROLLER7" (at 113.03 68.58 0)
       (effects (font (size 1.27 1.27)) hide)
     )
@@
     (instances
       (project "trinamic_wiring"
-        (path "/e4144788-6304-493f-818e-5d881d3b7418/c8eda2b5-ab13-4033-82d9-875c9fcaf884/13e2a7b5-46df-44bb-8dde-5d79d190b8bf"
-          (reference "MICROCONTROLLER4") (unit 1)
-        )
-        (path "/e4144788-6304-493f-818e-5d881d3b7418/c8eda2b5-ab13-4033-82d9-875c9fcaf884/e3613d8e-f506-47d6-ad2d-b0f5798d9847"
-          (reference "MICROCONTROLLER5") (unit 1)
-        )
         (path "/e4144788-6304-493f-818e-5d881d3b7418/c8eda2b5-ab13-4033-82d9-875c9fcaf884/5f6f310d-167d-42a3-8815-1b623fe73dc8"
           (reference "MICROCONTROLLER7") (unit 1)
         )
-        (path "/e4144788-6304-493f-818e-5d881d3b7418/c8eda2b5-ab13-4033-82d9-875c9fcaf884/00672f55-5cea-4051-abd7-9136695f76d0"
-          (reference "MICROCONTROLLER2") (unit 1)
+        (path "/e4144788-6304-493f-818e-5d881d3b7418/a161638e-a96f-4455-865a-1d7502675f43/5f6f310d-167d-42a3-8815-1b623fe73dc8"
+          (reference "MICROCONTROLLER4") (unit 1)
         )
       )

Commit message: Remove unused sheets
Parts:
- TMC11, TMC12: value DOC_TMC2209 -> TMC2209_DOC; symbol Janelia:DOC_TMC2209 -> Janelia:TMC2209_DOC
Changed lines of the file:
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@@
   (title_block
     (title "Trinamic Wiring")
-    (date "2023-08-02")
+    (date "2024-01-31")
     (rev "0.4")
     (company "Janelia Research Campus")
@@
     (effects (font (size 1.27 1.27)) (justify right bottom))
   )
-  (symbol (lib_name "DOC_TMC2209_1") (lib_id "Janelia:DOC_TMC2209") (at 166.37 87.63 0) (unit 1)
+  (symbol (lib_name "TMC2209_DOC_1") (lib_id "Janelia:TMC2209_DOC") (at 166.37 87.63 0) (unit 1)
     (in_bom yes) (on_board yes) (dnp no) (fields_autoplaced)
     (property "Reference" "TMC11" (at 166.37 68.58 0)
       (effects (font (size 1.27 1.27)) hide)
     )
-    (property "Value" "DOC_TMC2209" (at 166.37 73.66 0)
+    (property "Value" "TMC2209_DOC" (at 166.37 73.66 0)
       (effects (font (size 1.524 1.524)) hide)
     )
@@
           (reference "TMC11") (unit 1)
         )
-        (path "/e4144788-6304-493f-818e-5d881d3b7418/a161638e-a96f-4455-865a-1d7502675f43/5f6f310d-167d-42a3-8815-1b623fe73dc8"
-          (reference "TMC6") (unit 1)
-        )
       )
     )
   )
-  (symbol (lib_id "Janelia:DOC_TMC2209") (at 166.37 115.57 0) (unit 1)
+  (symbol (lib_id "Janelia:TMC2209_DOC") (at 166.37 115.57 0) (unit 1)
     (in_bom yes) (on_board yes) (dnp no) (fields_autoplaced)
     (property "Reference" "TMC12" (at 166.37 96.52 0)
       (effects (font (size 1.27 1.27)) hide)
     )
-    (property "Value" "DOC_TMC2209" (at 166.37 101.6 0)
+    (property "Value" "TMC2209_DOC" (at 166.37 101.6 0)
       (effects (font (size 1.524 1.524)) hide)
     )
@@
         (path "/e4144788-6304-493f-818e-5d881d3b7418/c8eda2b5-ab13-4033-82d9-875c9fcaf884/5f6f310d-167d-42a3-8815-1b623fe73dc8"
           (reference "TMC12") (unit 1)
-        )
-        (path "/e4144788-6304-493f-818e-5d881d3b7418/a161638e-a96f-4455-865a-1d7502675f43/5f6f310d-167d-42a3-8815-1b623fe73dc8"
-          (reference "TMC6") (unit 1)
         )
       )
@@
           (reference "R4") (unit 1)
         )
-        (path "/e4144788-6304-493f-818e-5d881d3b7418/a161638e-a96f-4455-865a-1d7502675f43/5f6f310d-167d-42a3-8815-1b623fe73dc8"
-          (reference "R2") (unit 1)
-        )
       )
     )
@@
           (reference "MICROCONTROLLER7") (unit 1)
         )
-        (path "/e4144788-6304-493f-818e-5d881d3b7418/a161638e-a96f-4455-865a-1d7502675f43/5f6f310d-167d-42a3-8815-1b623fe73dc8"
-          (reference "MICROCONTROLLER4") (unit 1)
-        )
       )
