File: trinamic_wiring/tmc2209_bidirectional_coupled_multiple_uart.kicad_sch (KiCad schematic)
At the start: 5 parts

Commit message: Remove unused sheets
Parts:
- TMC2, TMC3: value DOC_TMC2209 -> TMC2209_DOC; symbol Janelia:DOC_TMC2209 -> Janelia:TMC2209_DOC
Changed lines of the file:
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@@
   (title_block
     (title "Trinamic Wiring")
-    (date "2023-08-02")
+    (date "2024-01-31")
     (rev "0.4")
     (company "Janelia Research Campus")
@@
           (reference "R3") (unit 1)
         )
-        (path "/e4144788-6304-493f-818e-5d881d3b7418/a161638e-a96f-4455-865a-1d7502675f43/00672f55-5cea-4051-abd7-9136695f76d0"
-          (reference "R2") (unit 1)
-        )
       )
     )
@@
           (reference "R5") (unit 1)
         )
-        (path "/e4144788-6304-493f-818e-5d881d3b7418/a161638e-a96f-4455-865a-1d7502675f43/00672f55-5cea-4051-abd7-9136695f76d0"
-          (reference "R2") (unit 1)
-        )
-      )
-    )
-  )
-  (symbol (lib_id "Janelia:DOC_TMC2209") (at 162.56 116.84 0) (unit 1)
+      )
+    )
+  )
+  (symbol (lib_id "Janelia:TMC2209_DOC") (at 162.56 116.84 0) (unit 1)
     (in_bom yes) (on_board yes) (dnp no) (fields_autoplaced)
     (property "Reference" "TMC3" (at 162.56 97.79 0)
       (effects (font (size 1.27 1.27)) hide)
     )
-    (property "Value" "DOC_TMC2209" (at 162.56 102.87 0)
+    (property "Value" "TMC2209_DOC" (at 162.56 102.87 0)
       (effects (font (size 1.524 1.524)) hide)
     )
@@
           (reference "TMC3") (unit 1)
         )
-        (path "/e4144788-6304-493f-818e-5d881d3b7418/a161638e-a96f-4455-865a-1d7502675f43/00672f55-5cea-4051-abd7-9136695f76d0"
-          (reference "TMC6") (unit 1)
-        )
-      )
-    )
-  )
-  (symbol (lib_id "Janelia:DOC_TMC2209") (at 162.56 88.9 0) (unit 1)
+      )
+    )
+  )
+  (symbol (lib_id "Janelia:TMC2209_DOC") (at 162.56 88.9 0) (unit 1)
     (in_bom yes) (on_board yes) (dnp no) (fields_autoplaced)
     (property "Reference" "TMC2" (at 162.56 69.85 0)
       (effects (font (size 1.27 1.27)) hide)
     )
-    (property "Value" "DOC_TMC2209" (at 162.56 74.93 0)
+    (property "Value" "TMC2209_DOC" (at 162.56 74.93 0)
       (effects (font (size 1.524 1.524)) hide)
     )
@@
           (reference "TMC2") (unit 1)
         )
-        (path "/e4144788-6304-493f-818e-5d881d3b7418/a161638e-a96f-4455-865a-1d7502675f43/00672f55-5cea-4051-abd7-9136695f76d0"
-          (reference "TMC6") (unit 1)
-        )
       )
     )
@@
           (reference "MICROCONTROLLER2") (unit 1)
         )
-        (path "/e4144788-6304-493f-818e-5d881d3b7418/a161638e-a96f-4455-865a-1d7502675f43/00672f55-5cea-4051-abd7-9136695f76d0"
-          (reference "MICROCONTROLLER6") (unit 1)
-        )
-      )
+      )
