File: trinamic_wiring/tmc2209_description.kicad_sch (KiCad schematic)
At the start: 2 parts, among them M3 Stepper_Motor_QSH2818-32-07-0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

Commit message: Remove unused sheets
Parts:
- TMC13: value DOC_TMC2209 -> TMC2209_DOC; symbol Janelia:DOC_TMC2209 -> Janelia:TMC2209_DOC
Changed lines of the file:
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@@
   (title_block
     (title "Trinamic Wiring")
-    (date "2023-08-02")
+    (date "2024-01-31")
     (rev "0.4")
     (company "Janelia Research Campus")
@@
           (reference "M3") (unit 1)
         )
-        (path "/e4144788-6304-493f-818e-5d881d3b7418/a161638e-a96f-4455-865a-1d7502675f43/8277c47e-3fcc-48ef-9892-6d34b4c51a79"
-          (reference "M3") (unit 1)
-        )
       )
     )
   )
-  (symbol (lib_id "Janelia:DOC_TMC2209") (at 134.62 91.44 0) (unit 1)
+  (symbol (lib_id "Janelia:TMC2209_DOC") (at 134.62 91.44 0) (unit 1)
     (in_bom yes) (on_board yes) (dnp no) (fields_autoplaced)
     (property "Reference" "TMC13" (at 134.62 72.39 0)
       (effects (font (size 1.27 1.27)) hide)
     )
-    (property "Value" "DOC_TMC2209" (at 134.62 77.47 0)
+    (property "Value" "TMC2209_DOC" (at 134.62 77.47 0)
       (effects (font (size 1.524 1.524)) hide)
     )
@@
           (reference "TMC13") (unit 1)
         )
-        (path "/e4144788-6304-493f-818e-5d881d3b7418/a161638e-a96f-4455-865a-1d7502675f43/8277c47e-3fcc-48ef-9892-6d34b4c51a79"
-          (reference "TMC13") (unit 1)
-        )
