File: trinamic_wiring/tmc2209_stepper-controller.kicad_sch (KiCad schematic)
At the start: 8 parts, among them M5 Stepper_Motor_QSH2818-32-07-0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, M6 Stepper_Motor_QSH2818-32-07-0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, M7 Stepper_Motor_QSH2818-32-07-0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

Commit message: Remove unused sheets
Parts:
- TMC15, TMC17, TMC18: value DOC_TMC2209 -> TMC2209_DOC; symbol Janelia:DOC_TMC2209 -> Janelia:TMC2209_DOC
Changed lines of the file:
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@@
   (title_block
     (title "Trinamic Wiring")
-    (date "2023-08-02")
+    (date "2024-01-31")
     (rev "0.4")
     (company "Janelia Research Campus")
@@
     (effects (font (size 1.27 1.27)) (justify left bottom))
   )
-  (symbol (lib_id "Janelia:DOC_TMC2209") (at 144.78 129.54 0) (unit 1)
+  (symbol (lib_id "Janelia:TMC2209_DOC") (at 144.78 129.54 0) (unit 1)
     (in_bom yes) (on_board yes) (dnp no) (fields_autoplaced)
     (property "Reference" "TMC18" (at 144.78 110.49 0)
       (effects (font (size 1.27 1.27)) hide)
     )
-    (property "Value" "DOC_TMC2209" (at 144.78 115.57 0)
+    (property "Value" "TMC2209_DOC" (at 144.78 115.57 0)
       (effects (font (size 1.524 1.524)) hide)
     )
@@
           (reference "TMC18") (unit 1)
         )
-        (path "/e4144788-6304-493f-818e-5d881d3b7418/a161638e-a96f-4455-865a-1d7502675f43/262bc404-9876-4460-91a4-f9d4b0d72afb"
-          (reference "TMC18") (unit 1)
-        )
       )
     )
@@
           (reference "M5") (unit 1)
         )
-        (path "/e4144788-6304-493f-818e-5d881d3b7418/a161638e-a96f-4455-865a-1d7502675f43/262bc404-9876-4460-91a4-f9d4b0d72afb"
-          (reference "M3") (unit 1)
-        )
-      )
-    )
-  )
-  (symbol (lib_id "Janelia:DOC_TMC2209") (at 144.78 101.6 0) (unit 1)
+      )
+    )
+  )
+  (symbol (lib_id "Janelia:TMC2209_DOC") (at 144.78 101.6 0) (unit 1)
     (in_bom yes) (on_board yes) (dnp no) (fields_autoplaced)
     (property "Reference" "TMC17" (at 144.78 82.55 0)
       (effects (font (size 1.27 1.27)) hide)
     )
-    (property "Value" "DOC_TMC2209" (at 144.78 87.63 0)
+    (property "Value" "TMC2209_DOC" (at 144.78 87.63 0)
       (effects (font (size 1.524 1.524)) hide)
     )
@@
           (reference "TMC17") (unit 1)
         )
-        (path "/e4144788-6304-493f-818e-5d881d3b7418/a161638e-a96f-4455-865a-1d7502675f43/262bc404-9876-4460-91a4-f9d4b0d72afb"
-          (reference "TMC17") (unit 1)
-        )
       )
     )
@@
           (reference "TMC16") (unit 1)
         )
-        (path "/e4144788-6304-493f-818e-5d881d3b7418/a161638e-a96f-4455-865a-1d7502675f43/262bc404-9876-4460-91a4-f9d4b0d72afb"
-          (reference "TMC16") (unit 1)
-        )
-      )
-    )
-  )
-  (symbol (lib_id "Janelia:DOC_TMC2209") (at 144.78 73.66 0) (unit 1)
+      )
+    )
+  )
+  (symbol (lib_id "Janelia:TMC2209_DOC") (at 144.78 73.66 0) (unit 1)
     (in_bom yes) (on_board yes) (dnp no) (fields_autoplaced)
     (property "Reference" "TMC15" (at 144.78 54.61 0)
       (effects (font (size 1.27 1.27)) hide)
     )
-    (property "Value" "DOC_TMC2209" (at 144.78 59.69 0)
+    (property "Value" "TMC2209_DOC" (at 144.78 59.69 0)
       (effects (font (size 1.524 1.524)) hide)
     )
@@
           (reference "TMC15") (unit 1)
         )
-        (path "/e4144788-6304-493f-818e-5d881d3b7418/a161638e-a96f-4455-865a-1d7502675f43/262bc404-9876-4460-91a4-f9d4b0d72afb"
-          (reference "TMC15") (unit 1)
-        )
       )
     )
@@
           (reference "MICROCONTROLLER9") (unit 1)
         )
-        (path "/e4144788-6304-493f-818e-5d881d3b7418/a161638e-a96f-4455-865a-1d7502675f43/262bc404-9876-4460-91a4-f9d4b0d72afb"
-          (reference "MICROCONTROLLER9") (unit 1)
-        )
       )
     )
@@
           (reference "M7") (unit 1)
         )
-        (path "/e4144788-6304-493f-818e-5d881d3b7418/a161638e-a96f-4455-865a-1d7502675f43/262bc404-9876-4460-91a4-f9d4b0d72afb"
-          (reference "M3") (unit 1)
-        )
       )
     )
@@
           (reference "M6") (unit 1)
         )
-        (path "/e4144788-6304-493f-818e-5d881d3b7418/a161638e-a96f-4455-865a-1d7502675f43/262bc404-9876-4460-91a4-f9d4b0d72afb"
-          (reference "M3") (unit 1)
-        )
-      )
+      )
