File: trinamic_wiring/tmc2209_unidirectional_multiple.kicad_sch (KiCad schematic)
At the start: 3 parts

Commit message: Add TMC51X0 files
Parts:
- removed TMC6 (x2): DOC_TMC2209, symbol Janelia:DOC_TMC2209
- added TMC1, TMC8: DOC_TMC2209, symbol Janelia:DOC_TMC2209
- renumbered MICROCONTROLLER4 to MICROCONTROLLER1
Connections:
- net at MICROCONTROLLER1.1 (TX): now also TMC1.0 (UART), TMC8.0 (UART)
Changed lines of the file:
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@@
     (stroke (width 0) (type default))
   )
-  (symbol (lib_id "Janelia:DOC_MCU") (at 113.03 87.63 0) (unit 1)
+  (symbol (lib_id "Janelia:DOC_TMC2209") (at 163.83 115.57 0) (unit 1)
     (in_bom yes) (on_board yes) (dnp no) (fields_autoplaced)
-    (property "Reference" "MICROCONTROLLER4" (at 113.03 68.58 0)
+    (property "Reference" "TMC8" (at 163.83 96.52 0)
       (effects (font (size 1.27 1.27)) hide)
     )
-    (property "Value" "DOC_MCU" (at 113.03 73.66 0)
+    (property "Value" "DOC_TMC2209" (at 163.83 101.6 0)
       (effects (font (size 1.524 1.524)) hide)
     )
-    (property "Footprint" "" (at 110.49 114.3 0)
+    (property "Footprint" "" (at 161.29 142.24 0)
       (effects (font (size 1.524 1.524)) hide)
     )
-    (property "Datasheet" "" (at 113.03 87.63 0)
+    (property "Datasheet" "" (at 163.83 115.57 0)
       (effects (font (size 1.524 1.524)) hide)
     )
-    (property "Sim.Enable" "0" (at 113.03 71.12 0)
+    (property "Sim.Enable" "0" (at 163.83 99.06 0)
       (effects (font (size 1.27 1.27)) hide)
     )
     (pin "0")
     (pin "1")
+    (pin "10")
     (pin "2")
     (pin "3")
@@
     (pin "7")
     (pin "8")
+    (pin "9")
     (instances
       (project "trinamic_wiring"
-        (path "/e4144788-6304-493f-818e-5d881d3b7418/c8eda2b5-ab13-4033-82d9-875c9fcaf884/13e2a7b5-46df-44bb-8dde-5d79d190b8bf"
-          (reference "MICROCONTROLLER4") (unit 1)
+        (path "/e4144788-6304-493f-818e-5d881d3b7418/c8eda2b5-ab13-4033-82d9-875c9fcaf884/5b0a2695-6b0b-4c82-b9d6-7e19fee75501"
+          (reference "TMC8") (unit 1)
         )
-        (path "/e4144788-6304-493f-818e-5d881d3b7418/c8eda2b5-ab13-4033-82d9-875c9fcaf884/5b0a2695-6b0b-4c82-b9d6-7e19fee75501"
-          (reference "MICROCONTROLLER1") (unit 1)
-        )
-        (path "/e4144788-6304-493f-818e-5d881d3b7418/c8eda2b5-ab13-4033-82d9-875c9fcaf884/d4a56977-1958-4e49-bd54-bb12e595a31d"
-          (reference "MICROCONTROLLER6") (unit 1)
+        (path "/e4144788-6304-493f-818e-5d881d3b7418/a161638e-a96f-4455-865a-1d7502675f43/5b0a2695-6b0b-4c82-b9d6-7e19fee75501"
+          (reference "TMC6") (unit 1)
         )
       )
@@
   (symbol (lib_id "Janelia:DOC_TMC2209") (at 163.83 87.63 0) (unit 1)
     (in_bom yes) (on_board yes) (dnp no) (fields_autoplaced)
-    (property "Reference" "TMC6" (at 163.83 68.58 0)
+    (property "Reference" "TMC1" (at 163.83 68.58 0)
       (effects (font (size 1.27 1.27)) hide)
     )
@@
     (instances
       (project "trinamic_wiring"
-        (path "/e4144788-6304-493f-818e-5d881d3b7418/c8eda2b5-ab13-4033-82d9-875c9fcaf884/13e2a7b5-46df-44bb-8dde-5d79d190b8bf"
-          (reference "TMC6") (unit 1)
-        )
         (path "/e4144788-6304-493f-818e-5d881d3b7418/c8eda2b5-ab13-4033-82d9-875c9fcaf884/5b0a2695-6b0b-4c82-b9d6-7e19fee75501"
           (reference "TMC1") (unit 1)
         )
-        (path "/e4144788-6304-493f-818e-5d881d3b7418/c8eda2b5-ab13-4033-82d9-875c9fcaf884/d4a56977-1958-4e49-bd54-bb12e595a31d"
-          (reference "TMC9") (unit 1)
+        (path "/e4144788-6304-493f-818e-5d881d3b7418/a161638e-a96f-4455-865a-1d7502675f43/5b0a2695-6b0b-4c82-b9d6-7e19fee75501"
+          (reference "TMC6") (unit 1)
         )
       )
     )
   )
-  (symbol (lib_id "Janelia:DOC_TMC2209") (at 163.83 115.57 0) (unit 1)
+  (symbol (lib_id "Janelia:DOC_MCU") (at 113.03 87.63 0) (unit 1)
     (in_bom yes) (on_board yes) (dnp no) (fields_autoplaced)
-    (property "Reference" "TMC6" (at 163.83 96.52 0)
+    (property "Reference" "MICROCONTROLLER1" (at 113.03 68.58 0)
       (effects (font (size 1.27 1.27)) hide)
     )
-    (property "Value" "DOC_TMC2209" (at 163.83 101.6 0)
+    (property "Value" "DOC_MCU" (at 113.03 73.66 0)
       (effects (font (size 1.524 1.524)) hide)
     )
-    (property "Footprint" "" (at 161.29 142.24 0)
+    (property "Footprint" "" (at 110.49 114.3 0)
       (effects (font (size 1.524 1.524)) hide)
     )
-    (property "Datasheet" "" (at 163.83 115.57 0)
+    (property "Datasheet" "" (at 113.03 87.63 0)
       (effects (font (size 1.524 1.524)) hide)
     )
-    (property "Sim.Enable" "0" (at 163.83 99.06 0)
+    (property "Sim.Enable" "0" (at 113.03 71.12 0)
       (effects (font (size 1.27 1.27)) hide)
     )
     (pin "0")
     (pin "1")
-    (pin "10")
     (pin "2")
     (pin "3")
@@
     (pin "7")
     (pin "8")
-    (pin "9")
     (instances
       (project "trinamic_wiring"
-        (path "/e4144788-6304-493f-818e-5d881d3b7418/c8eda2b5-ab13-4033-82d9-875c9fcaf884/13e2a7b5-46df-44bb-8dde-5d79d190b8bf"
-          (reference "TMC6") (unit 1)
+        (path "/e4144788-6304-493f-818e-5d881d3b7418/c8eda2b5-ab13-4033-82d9-875c9fcaf884/5b0a2695-6b0b-4c82-b9d6-7e19fee75501"
+          (reference "MICROCONTROLLER1") (unit 1)
         )
-        (path "/e4144788-6304-493f-818e-5d881d3b7418/c8eda2b5-ab13-4033-82d9-875c9fcaf884/5b0a2695-6b0b-4c82-b9d6-7e19fee75501"
-          (reference "TMC8") (unit 1)
-        )
-        (path "/e4144788-6304-493f-818e-5d881d3b7418/c8eda2b5-ab13-4033-82d9-875c9fcaf884/d4a56977-1958-4e49-bd54-bb12e595a31d"
-          (reference "TMC10") (unit 1)
+        (path "/e4144788-6304-493f-818e-5d881d3b7418/a161638e-a96f-4455-865a-1d7502675f43/5b0a2695-6b0b-4c82-b9d6-7e19fee75501"
+          (reference "MICROCONTROLLER4") (unit 1)
         )
       )

Commit message: Remove unused sheets
Parts:
- TMC1, TMC8: value DOC_TMC2209 -> TMC2209_DOC; symbol Janelia:DOC_TMC2209 -> Janelia:TMC2209_DOC
Changed lines of the file:
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@@
   (title_block
     (title "Trinamic Wiring")
-    (date "2023-08-02")
+    (date "2024-01-31")
     (rev "0.4")
     (company "Janelia Research Campus")
@@
     (stroke (width 0) (type default))
   )
-  (symbol (lib_id "Janelia:DOC_TMC2209") (at 163.83 115.57 0) (unit 1)
+  (symbol (lib_id "Janelia:TMC2209_DOC") (at 163.83 115.57 0) (unit 1)
     (in_bom yes) (on_board yes) (dnp no) (fields_autoplaced)
     (property "Reference" "TMC8" (at 163.83 96.52 0)
       (effects (font (size 1.27 1.27)) hide)
     )
-    (property "Value" "DOC_TMC2209" (at 163.83 101.6 0)
+    (property "Value" "TMC2209_DOC" (at 163.83 101.6 0)
       (effects (font (size 1.524 1.524)) hide)
     )
@@
           (reference "TMC8") (unit 1)
         )
-        (path "/e4144788-6304-493f-818e-5d881d3b7418/a161638e-a96f-4455-865a-1d7502675f43/5b0a2695-6b0b-4c82-b9d6-7e19fee75501"
-          (reference "TMC6") (unit 1)
-        )
       )
     )
   )
-  (symbol (lib_id "Janelia:DOC_TMC2209") (at 163.83 87.63 0) (unit 1)
+  (symbol (lib_id "Janelia:TMC2209_DOC") (at 163.83 87.63 0) (unit 1)
     (in_bom yes) (on_board yes) (dnp no) (fields_autoplaced)
     (property "Reference" "TMC1" (at 163.83 68.58 0)
       (effects (font (size 1.27 1.27)) hide)
     )
-    (property "Value" "DOC_TMC2209" (at 163.83 73.66 0)
+    (property "Value" "TMC2209_DOC" (at 163.83 73.66 0)
       (effects (font (size 1.524 1.524)) hide)
     )
@@
         (path "/e4144788-6304-493f-818e-5d881d3b7418/c8eda2b5-ab13-4033-82d9-875c9fcaf884/5b0a2695-6b0b-4c82-b9d6-7e19fee75501"
           (reference "TMC1") (unit 1)
-        )
-        (path "/e4144788-6304-493f-818e-5d881d3b7418/a161638e-a96f-4455-865a-1d7502675f43/5b0a2695-6b0b-4c82-b9d6-7e19fee75501"
-          (reference "TMC6") (unit 1)
         )
       )
@@
           (reference "MICROCONTROLLER1") (unit 1)
         )
-        (path "/e4144788-6304-493f-818e-5d881d3b7418/a161638e-a96f-4455-865a-1d7502675f43/5b0a2695-6b0b-4c82-b9d6-7e19fee75501"
-          (reference "MICROCONTROLLER4") (unit 1)
-        )
       )
