File: trinamic_wiring/tmc2209_unidirectional_multiple_uart.kicad_sch (KiCad schematic)
At the start: 3 parts

Commit message: Add TMC51X0 files
Parts:
- renumbered TMC6 to TMC10, TMC6 to TMC9
Changed lines of the file:
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@@
+          (reference "MICROCONTROLLER6") (unit 1)
+        )
+        (path "/e4144788-6304-493f-818e-5d881d3b7418/a161638e-a96f-4455-865a-1d7502675f43/d4a56977-1958-4e49-bd54-bb12e595a31d"
           (reference "MICROCONTROLLER6") (unit 1)
         )
@@
   (symbol (lib_id "Janelia:DOC_TMC2209") (at 163.83 87.63 0) (unit 1)
     (in_bom yes) (on_board yes) (dnp no) (fields_autoplaced)
-    (property "Reference" "TMC6" (at 163.83 68.58 0)
+    (property "Reference" "TMC9" (at 163.83 68.58 0)
       (effects (font (size 1.27 1.27)) hide)
     )
@@
     (instances
       (project "trinamic_wiring"
-        (path "/e4144788-6304-493f-818e-5d881d3b7418/c8eda2b5-ab13-4033-82d9-875c9fcaf884/13e2a7b5-46df-44bb-8dde-5d79d190b8bf"
-          (reference "TMC6") (unit 1)
-        )
-        (path "/e4144788-6304-493f-818e-5d881d3b7418/c8eda2b5-ab13-4033-82d9-875c9fcaf884/5b0a2695-6b0b-4c82-b9d6-7e19fee75501"
-          (reference "TMC1") (unit 1)
-        )
         (path "/e4144788-6304-493f-818e-5d881d3b7418/c8eda2b5-ab13-4033-82d9-875c9fcaf884/d4a56977-1958-4e49-bd54-bb12e595a31d"
           (reference "TMC9") (unit 1)
+        )
+        (path "/e4144788-6304-493f-818e-5d881d3b7418/a161638e-a96f-4455-865a-1d7502675f43/d4a56977-1958-4e49-bd54-bb12e595a31d"
+          (reference "TMC6") (unit 1)
         )
       )
@@
   (symbol (lib_id "Janelia:DOC_TMC2209") (at 163.83 115.57 0) (unit 1)
     (in_bom yes) (on_board yes) (dnp no) (fields_autoplaced)
-    (property "Reference" "TMC6" (at 163.83 96.52 0)
+    (property "Reference" "TMC10" (at 163.83 96.52 0)
       (effects (font (size 1.27 1.27)) hide)
     )
@@
     (instances
       (project "trinamic_wiring"
-        (path "/e4144788-6304-493f-818e-5d881d3b7418/c8eda2b5-ab13-4033-82d9-875c9fcaf884/13e2a7b5-46df-44bb-8dde-5d79d190b8bf"
-          (reference "TMC6") (unit 1)
-        )
-        (path "/e4144788-6304-493f-818e-5d881d3b7418/c8eda2b5-ab13-4033-82d9-875c9fcaf884/5b0a2695-6b0b-4c82-b9d6-7e19fee75501"
-          (reference "TMC8") (unit 1)
-        )
         (path "/e4144788-6304-493f-818e-5d881d3b7418/c8eda2b5-ab13-4033-82d9-875c9fcaf884/d4a56977-1958-4e49-bd54-bb12e595a31d"
           (reference "TMC10") (unit 1)
         )
+        (path "/e4144788-6304-493f-818e-5d881d3b7418/a161638e-a96f-4455-865a-1d7502675f43/d4a56977-1958-4e49-bd54-bb12e595a31d"
+          (reference "TMC6") (unit 1)
+        )
       )

Commit message: Remove unused sheets
Parts:
- TMC10, TMC9: value DOC_TMC2209 -> TMC2209_DOC; symbol Janelia:DOC_TMC2209 -> Janelia:TMC2209_DOC
Changed lines of the file:
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@@
   (title_block
     (title "Trinamic Wiring")
-    (date "2023-08-02")
+    (date "2024-01-31")
     (rev "0.4")
     (company "Janelia Research Campus")
@@
           (reference "MICROCONTROLLER6") (unit 1)
         )
-        (path "/e4144788-6304-493f-818e-5d881d3b7418/a161638e-a96f-4455-865a-1d7502675f43/d4a56977-1958-4e49-bd54-bb12e595a31d"
-          (reference "MICROCONTROLLER6") (unit 1)
-        )
       )
     )
   )
-  (symbol (lib_id "Janelia:DOC_TMC2209") (at 163.83 87.63 0) (unit 1)
+  (symbol (lib_id "Janelia:TMC2209_DOC") (at 163.83 87.63 0) (unit 1)
     (in_bom yes) (on_board yes) (dnp no) (fields_autoplaced)
     (property "Reference" "TMC9" (at 163.83 68.58 0)
       (effects (font (size 1.27 1.27)) hide)
     )
-    (property "Value" "DOC_TMC2209" (at 163.83 73.66 0)
+    (property "Value" "TMC2209_DOC" (at 163.83 73.66 0)
       (effects (font (size 1.524 1.524)) hide)
     )
@@
           (reference "TMC9") (unit 1)
         )
-        (path "/e4144788-6304-493f-818e-5d881d3b7418/a161638e-a96f-4455-865a-1d7502675f43/d4a56977-1958-4e49-bd54-bb12e595a31d"
-          (reference "TMC6") (unit 1)
-        )
       )
     )
   )
-  (symbol (lib_id "Janelia:DOC_TMC2209") (at 163.83 115.57 0) (unit 1)
+  (symbol (lib_id "Janelia:TMC2209_DOC") (at 163.83 115.57 0) (unit 1)
     (in_bom yes) (on_board yes) (dnp no) (fields_autoplaced)
     (property "Reference" "TMC10" (at 163.83 96.52 0)
       (effects (font (size 1.27 1.27)) hide)
     )
-    (property "Value" "DOC_TMC2209" (at 163.83 101.6 0)
+    (property "Value" "TMC2209_DOC" (at 163.83 101.6 0)
       (effects (font (size 1.524 1.524)) hide)
     )
@@
           (reference "TMC10") (unit 1)
         )
-        (path "/e4144788-6304-493f-818e-5d881d3b7418/a161638e-a96f-4455-865a-1d7502675f43/d4a56977-1958-4e49-bd54-bb12e595a31d"
-          (reference "TMC6") (unit 1)
-        )
       )
